Commit message: urdf modified

File: src/myagv_description/urdf/agv.urdf (robot description, URDF)
Before this commit: robot agv, 7 links, 6 joints
Joints:
- joint base_joint: child base_link -> base_footprint; origin xyz=0.0 0.0 0.01 rpy=0.0 0.0 0.0 -> xyz=0.0 0.0 0.17181 rpy=0.0 0.0 0.0; parent base_footprint -> base_link
- joint dummy_joint: child base_footprint -> base_link
- joint lidar_joint: origin xyz=-0.035 -0.035 0.2025 rpy=0.0 0.0 0.0 -> xyz=-0.165 0.07 0.12 rpy=0.0 0.0 -1.57
- joint wheel_left_joint: origin xyz=-0.077 0.125 0.07967 rpy=0.0 0.0 0.0 -> xyz=0.0 0.17 0.02 rpy=0.0 0.0 0.0
- joint wheel_right_joint: origin xyz=-0.077 -0.125 0.07967 rpy=0.0 0.0 3.14 -> xyz=0.0 -0.17 0.02 rpy=0.0 0.0 3.14
